Commit message: LiDAR Update

File: rugved_description/urdf/rugved_description.urdf (robot description, URDF)
Before this commit: robot rugved_description, 5 links, 4 joints
Links:
- added link hokuyo_link, mass 1e-5; collision box size=0.1 0.1 0.1; visual box size=0.1 0.1 0.1
Joints:
- added joint hokuyo_joint: type fixed, parent base_link, child hokuyo_link, origin xyz=-0.55 0.0 0.55 rpy=0 0 3.14, axis 0 1 0

Commit message: Camera Update

File: rugved_description/urdf/rugved_description.urdf (robot description, URDF)
Before this commit: robot rugved_description, 6 links, 5 joints
Links:
- added link camera_link, mass 1e-5; collision box size=0.1 0.1 0.1; visual box size=0.1 0.1 0.1
Joints:
- added joint camera_joint: type fixed, parent base_link, child camera_link, origin xyz=-0.60025 -0.00023509 0.55 rpy=0 0 3.14, axis 0 1 0
- joint hokuyo_joint: origin xyz=-0.55 0.0 0.55 rpy=0 0 3.14 -> xyz=0.10025 -0.00023509 0.74914 rpy=0 0 3.14

Commit message: Visual for GPS and IMU; Joint Values fixed.

File: rugved_description/urdf/rugved_description.urdf (robot description, URDF)
Before this commit: robot rugved_description, 7 links, 6 joints
Links:
- added link gps_link, mass 1e-5; collision box size=0.03 0.05 0.01; visual box size=0.03 0.05 0.01
- added link imu_link, mass 1e-5; collision box size=0.03 0.05 0.01; visual box size=0.03 0.05 0.01
Joints:
- added joint gps_joint: type fixed, parent base_link, child gps_link, origin xyz=0.07525 -0.00023509 0.24914 rpy=0 0 0, axis 0 1 0
- added joint imu_joint: type fixed, parent base_link, child imu_link, origin xyz=0.12525 -0.00023509 0.24914 rpy=0 0 0, axis 0 1 0
- joint horizontal_castor_joint: limit lower=0 upper=6.29 effort=500 velocity=1 -> lower=-1000000 upper=1000000 effort=500 velocity=1
- joint left_wheel_joint: limit lower=0 upper=6.29 effort=1000 velocity=1 -> lower=-1000000 upper=1000000 effort=1000 velocity=1
- joint right_wheel_joint: limit lower=0 upper=6.29 effort=1000 velocity=1 -> lower=-1000000 upper=1000000 effort=1000 velocity=1
- joint vertical_castor_joint: limit lower=0 upper=6.29 effort=400 velocity=1 -> lower=-1000000 upper=1000000 effort=400 velocity=1
